Commit message: Add: chandra gazebo package

File: src/chandra_description/urdf/chandra_arm.urdf.xacro (robot description, xacro)
@@ -2,11 +2,16 @@
 <robot name="dofbot">
     <link name="base_link">
-        <visual>
-            <origin
-                    xyz="0 0 0"
-                    rpy="0 0 0"/>
-            <geometry>
-                <mesh
-                        filename="package://chandra_description/meshes/base_link.STL"/>
+        <inertial>
+            <origin xyz="0 0 0" rpy="0 0 0"/>
+            <mass value="0.1"/>
+            <inertia ixx="0.0001" ixy="0.0" ixz="0.0" iyy="0.0001" iyz="0.0" izz="0.0001"/>
+        </inertial>
+        <visual>
+            <origin
+                    xyz="0 0 0"
+                    rpy="0 0 0"/>
+            <geometry>
+                <mesh
+                        filename="file://$(find chandra_description)/meshes/base_link.STL"/>
             </geometry>
             <material
@@ -22,16 +27,21 @@
             <geometry>
                 <mesh
-                        filename="package://chandra_description/meshes/base_link.STL"/>
+                        filename="file://$(find chandra_description)/meshes/base_link.STL"/>
             </geometry>
         </collision>
     </link>
     <link name="link1">
-        <visual>
-            <origin
-                    xyz="0 0 0"
-                    rpy="0 0 0"/>
-            <geometry>
-                <mesh
-                        filename="package://chandra_description/meshes/link1.STL"/>
+        <inertial>
+            <origin xyz="0 0 0" rpy="0 0 0"/>
+            <mass value="0.1"/>
+            <inertia ixx="0.0001" ixy="0.0" ixz="0.0" iyy="0.0001" iyz="0.0" izz="0.0001"/>
+        </inertial>
+        <visual>
+            <origin
+                    xyz="0 0 0"
+                    rpy="0 0 0"/>
+            <geometry>
+                <mesh
+                        filename="file://$(find chandra_description)/meshes/link1.STL"/>
             </geometry>
             <material
@@ -47,5 +57,5 @@
             <geometry>
                 <mesh
-                        filename="package://chandra_description/meshes/link1.STL"/>
+                        filename="file://$(find chandra_description)/meshes/link1.STL"/>
             </geometry>
         </collision>
@@ -68,11 +78,16 @@
     </joint>
     <link name="link2">
-        <visual>
-            <origin
-                    xyz="0 0 0"
-                    rpy="0 0 0"/>
-            <geometry>
-                <mesh
-                        filename="package://chandra_description/meshes/link2.STL"/>
+        <inertial>
+            <origin xyz="0 0 0" rpy="0 0 0"/>
+            <mass value="0.1"/>
+            <inertia ixx="0.0001" ixy="0.0" ixz="0.0" iyy="0.0001" iyz="0.0" izz="0.0001"/>
+        </inertial>
+        <visual>
+            <origin
+                    xyz="0 0 0"
+                    rpy="0 0 0"/>
+            <geometry>
+                <mesh
+                        filename="file://$(find chandra_description)/meshes/link2.STL"/>
             </geometry>
             <material
@@ -88,5 +103,5 @@
             <geometry>
                 <mesh
-                        filename="package://chandra_description/meshes/link2.STL"/>
+                        filename="file://$(find chandra_description)/meshes/link2.STL"/>
             </geometry>
         </collision>
@@ -109,11 +124,16 @@
     </joint>
     <link name="link3">
-        <visual>
-            <origin
-                    xyz="0 0 0"
-                    rpy="0 0 0"/>
-            <geometry>
-                <mesh
-                        filename="package://chandra_description/meshes/link3.STL"/>
+        <inertial>
+            <origin xyz="0 0 0" rpy="0 0 0"/>
+            <mass value="0.1"/>
+            <inertia ixx="0.0001" ixy="0.0" ixz="0.0" iyy="0.0001" iyz="0.0" izz="0.0001"/>
+        </inertial>
+        <visual>
+            <origin
+                    xyz="0 0 0"
+                    rpy="0 0 0"/>
+            <geometry>
+                <mesh
+                        filename="file://$(find chandra_description)/meshes/link3.STL"/>
             </geometry>
             <material
@@ -129,5 +149,5 @@
             <geometry>
                 <mesh
-                        filename="package://chandra_description/meshes/link3.STL"/>
+                        filename="file://$(find chandra_description)/meshes/link3.STL"/>
             </geometry>
         </collision>
@@ -150,11 +170,16 @@
     </joint>
     <link name="link4">
-        <visual>
-            <origin
-                    xyz="0 0 0"
-                    rpy="0 0 0"/>
-            <geometry>
-                <mesh
-                        filename="package://chandra_description/meshes/link4.STL"/>
+        <inertial>
+            <origin xyz="0 0 0" rpy="0 0 0"/>
+            <mass value="0.1"/>
+            <inertia ixx="0.0001" ixy="0.0" ixz="0.0" iyy="0.0001" iyz="0.0" izz="0.0001"/>
+        </inertial>
+        <visual>
+            <origin
+                    xyz="0 0 0"
+                    rpy="0 0 0"/>
+            <geometry>
+                <mesh
+                        filename="file://$(find chandra_description)/meshes/link4.STL"/>
             </geometry>
             <material
@@ -170,5 +195,5 @@
             <geometry>
                 <mesh
-                        filename="package://chandra_description/meshes/link4.STL"/>
+                        filename="file://$(find chandra_description)/meshes/link4.STL"/>
             </geometry>
         </collision>
@@ -191,11 +216,16 @@
     </joint>
     <link name="link5">
-        <visual>
-            <origin
-                    xyz="0 0 0"
-                    rpy="0 0 0"/>
-            <geometry>
-                <mesh
-                        filename="package://chandra_description/meshes/link5.STL"/>
+        <inertial>
+            <origin xyz="0 0 0" rpy="0 0 0"/>
+            <mass value="0.1"/>
+            <inertia ixx="0.0001" ixy="0.0" ixz="0.0" iyy="0.0001" iyz="0.0" izz="0.0001"/>
+        </inertial>
+        <visual>
+            <origin
+                    xyz="0 0 0"
+                    rpy="0 0 0"/>
+            <geometry>
+                <mesh
+                        filename="file://$(find chandra_description)/meshes/link5.STL"/>
             </geometry>
             <material
@@ -211,5 +241,5 @@
             <geometry>
                 <mesh
-                        filename="package://chandra_description/meshes/link5.STL"/>
+                        filename="file://$(find chandra_description)/meshes/link5.STL"/>
             </geometry>
         </collision>

Commit message: Add chandra control package

File: src/chandra_description/urdf/chandra_arm.urdf.xacro (robot description, xacro)
@@ -1,4 +1,20 @@
 <?xml version="1.0" encoding="utf-8"?>
-<robot name="dofbot">
+<robot name="chandra" xmlns:xacro="http://www.ros.org/wiki/xacro">
+    <xacro:property name="effort" value="100"/>
+    <xacro:property name="velocity" value="1"/>
+    <!-- Useful Macros -->
+    <xacro:macro name="default_inertial" params="mass">
+        <inertial>
+            <origin xyz="0 0 0" rpy="0 0 0"/>
+            <mass value="${mass}" />
+            <inertia ixx="1.0" ixy="0.0" ixz="0.0"
+                     iyy="1.0" iyz="0.0"
+                     izz="1.0" />
+        </inertial>
+    </xacro:macro>
+    <!-- Include Gazebo Parameters -->
+    <xacro:include filename="$(find chandra_description)/urdf/chandra_arm_gazebo.xacro" />
+    <!-- Include ros2_control Plugins -->
+    <xacro:include filename="$(find chandra_description)/urdf/chandra_arm_control.xacro" />
     <link name="base_link">
         <inertial>
@@ -74,6 +90,6 @@
                 lower="-1.5708"
                 upper="1.5708"
-                effort="100"
-                velocity="1"/>
+                effort="${effort}"
+                velocity="${velocity}"/>
     </joint>
     <link name="link2">
@@ -120,6 +136,6 @@
                 lower="-1.5708"
                 upper="1.5708"
-                effort="100"
-                velocity="1"/>
+                effort="${effort}"
+                velocity="${velocity}"/>
     </joint>
     <link name="link3">
@@ -166,6 +182,6 @@
                 lower="-1.5708"
                 upper="1.5708"
-                effort="100"
-                velocity="1"/>
+                effort="${effort}"
+                velocity="${velocity}"/>
     </joint>
     <link name="link4">
@@ -212,6 +228,6 @@
                 lower="-1.5708"
                 upper="1.5708"
-                effort="100"
-                velocity="1"/>
+                effort="${effort}"
+                velocity="${velocity}"/>
     </joint>
     <link name="link5">
@@ -258,6 +274,65 @@
                 lower="-1.5708"
                 upper="3.1416"
-                effort="100"
-                velocity="1"/>
+                effort="${effort}"
+                velocity="${velocity}"/>
+    </joint>
+    <link name="gripper_right">
+        <xacro:default_inertial mass="0.01"/>
+        <visual>
+            <origin
+                    xyz="0 0 0"
+                    rpy="0 0 0"/>
+            <geometry>
+                <mesh filename="file://$(find chandra_description)/meshes/gripper_right_finger.STL"/>
+            </geometry>
+        </visual>
+        <collision>
+            <origin
+                    xyz="0 0 0"
+                    rpy="0 0 0"/>
+            <geometry>
+                <mesh filename="file://$(find chandra_description)/meshes/gripper_right_finger.STL"/>
+            </geometry>
+        </collision>
+    </link>
+    <joint name ="joint_6" type="revolute">
+        <parent link="link5"/>
+        <child link = "gripper_right"/>
+        <origin
+                xyz="0 0 0"
+                rpy="0 0 0"/>
+        <axis xyz="0 0 1"/>
+        <limit lower="-${PI / 2}" upper="0.0"
+               effort="${effort}" velocity="${velocity}"/>
+    </joint>
+    <link name="gripper_left">
+        <xacro:default_inertial mass="0.01"/>
+        <visual>
+            <origin
+                    xyz="0 0 0"
+                    rpy="0 0 0"/>
+            <geometry>
+                <mesh filename="file://$(find chandra_description)/meshes/gripper_left_finger.STL"/>
+            </geometry>
+        </visual>
+        <collision>
+            <origin
+                    xyz="0 0 0"
+                    rpy="0 0 0"/>
+            <geometry>
+                <mesh filename="file://$(find chandra_description)/meshes/gripper_left_finger.STL"/>
+            </geometry>
+        </collision>
+    </link>
+    <joint name ="joint_7" type="revolute">
+        <parent link="link5"/>
+        <child link = "gripper_left"/>
+        <origin
+                xyz="0 0 0"
+                rpy="0 0 0"/>
+        <axis xyz="0 0 1"/>
+        <limit lower="0.0" upper="${PI / 2}"
+               effort="${effort}" velocity="${velocity}"/>
+        <mimic joint="joint_6" multiplier="-1"/>
     </joint>
 </robot>

Commit message: Update: chandra control package

File: src/chandra_description/urdf/chandra_arm.urdf.xacro (robot description, xacro)
@@ -281,5 +281,5 @@
         <visual>
             <origin
-                    xyz="0 0 0"
+                    xyz="0.0121 0 -0.0335"
                     rpy="0 0 0"/>
             <geometry>
@@ -289,5 +289,5 @@
         <collision>
             <origin
-                    xyz="0 0 0"
+                    xyz="0.0121 0 -0.0335"
                     rpy="0 0 0"/>
             <geometry>
@@ -296,11 +296,11 @@
         </collision>
     </link>
-    <joint name ="joint_6" type="revolute">
+    <joint name ="joint6" type="revolute">
         <parent link="link5"/>
         <child link = "gripper_right"/>
         <origin
-                xyz="0 0 0"
-                rpy="0 0 0"/>
-        <axis xyz="0 0 1"/>
+                xyz="-0.0121 0 0.0335"
+                rpy="0 0 0"/>
+        <axis xyz="0 1 0"/>
         <limit lower="-${PI / 2}" upper="0.0"
                effort="${effort}" velocity="${velocity}"/>
@@ -310,5 +310,5 @@
         <visual>
             <origin
-                    xyz="0 0 0"
+                    xyz="-0.0121 0 -0.0335"
                     rpy="0 0 0"/>
             <geometry>
@@ -318,5 +318,5 @@
         <collision>
             <origin
-                    xyz="0 0 0"
+                    xyz="-0.0121 0 -0.0335"
                     rpy="0 0 0"/>
             <geometry>
@@ -325,14 +325,14 @@
         </collision>
     </link>
-    <joint name ="joint_7" type="revolute">
+    <joint name ="joint7" type="revolute">
         <parent link="link5"/>
         <child link = "gripper_left"/>
         <origin
-                xyz="0 0 0"
-                rpy="0 0 0"/>
-        <axis xyz="0 0 1"/>
+                xyz="0.0121 0 0.0335"
+                rpy="0 0 0"/>
+        <axis xyz="0 1 0"/>
         <limit lower="0.0" upper="${PI / 2}"
                effort="${effort}" velocity="${velocity}"/>
-        <mimic joint="joint_6" multiplier="-1"/>
+        <mimic joint="joint6" multiplier="-1"/>
     </joint>
 </robot>

File: src/chandra_description/urdf/chandra_arm_control.xacro (robot description, xacro)
@@ -6,5 +6,5 @@
             <plugin>gz_ros2_control/GazeboSimSystem</plugin>
         </hardware>
-        <joint name="joint_1">
+        <joint name="joint1">
             <command_interface name="position">
             <param name="min">-${PI / 2}</param>
@@ -13,5 +13,5 @@
             <state_interface name="position"/>
         </joint>
-        <joint name="joint_2">
+        <joint name="joint2">
             <command_interface name="position">
             <param name="min">-${PI / 2}</param>
@@ -20,5 +20,5 @@
             <state_interface name="position"/>
         </joint>
-        <joint name="joint_3">
+        <joint name="joint3">
             <command_interface name="position">
             <param name="min">-${PI / 2}</param>
@@ -27,5 +27,5 @@
             <state_interface name="position"/>
         </joint>
-        <joint name="joint_4">
+        <joint name="joint4">
             <command_interface name="position">
             <param name="min">-${PI / 2}</param>
@@ -34,5 +34,5 @@
             <state_interface name="position"/>
         </joint>
-        <joint name="joint_5">
+        <joint name="joint5">
             <command_interface name="position">
             <param name="min">-${PI / 2}</param>
@@ -41,5 +41,5 @@
             <state_interface name="position"/>
         </joint>
-        <joint name="joint_6">
+        <joint name="joint6">
             <command_interface name="position">
             <param name="min">-${PI / 2}</param>
@@ -48,6 +48,6 @@
             <state_interface name="position"/>
         </joint>
-        <joint name="joint_7">
-            <param name="mimic">joint_6</param>
+        <joint name="joint7">
+            <param name="mimic">joint6</param>
             <param name="multiplier">-1</param>
         </joint>
