Commit message: Complete: chandra control package

File: src/chandra_description/urdf/chandra_arm.urdf.xacro (robot description, xacro)
@@ -1,4 +1,18 @@
 <?xml version="1.0" encoding="utf-8"?>
 <robot name="chandra" xmlns:xacro="http://www.ros.org/wiki/xacro">
+        <!-- Color Properties -->
+        <xacro:property name="deep_blue" value="0.0 0.0 0.6 1"/>
+        <xacro:property name="green" value="0.0 0.7 0.0 1"/>
+        <xacro:property name="black" value="0.05 0.05 0.05 1"/>
+        <!-- Macro for metallic material -->
+        <xacro:macro name="metallic_material" params="name colour">
+                <material name="${name}">
+                        <color rgba="${colour}"/>
+                        <specular value="0.8 0.8 0.8 1"/>
+                </material>
+        </xacro:macro>
+        <!-- Xacro Properties for common values -->
+        <xacro:property name="default_colour" value="0.7 0.7 0.7 1"/>
+        <xacro:property name="default_scale" value="1 1 1"/>
     <xacro:property name="effort" value="100"/>
     <xacro:property name="velocity" value="1"/>
@@ -18,60 +32,38 @@
     <xacro:include filename="$(find chandra_description)/urdf/chandra_arm_control.xacro" />
     <link name="base_link">
-        <inertial>
-            <origin xyz="0 0 0" rpy="0 0 0"/>
-            <mass value="0.1"/>
-            <inertia ixx="0.0001" ixy="0.0" ixz="0.0" iyy="0.0001" iyz="0.0" izz="0.0001"/>
-        </inertial>
-        <visual>
-            <origin
-                    xyz="0 0 0"
-                    rpy="0 0 0"/>
-            <geometry>
-                <mesh
-                        filename="file://$(find chandra_description)/meshes/base_link.STL"/>
-            </geometry>
-            <material
-                    name="">
-                <color
-                        rgba="0.7 0.7 0.7 1"/>
-            </material>
-        </visual>
-        <collision>
-            <origin
-                    xyz="0 0 0"
-                    rpy="0 0 0"/>
-            <geometry>
-                <mesh
-                        filename="file://$(find chandra_description)/meshes/base_link.STL"/>
+        <xacro:default_inertial mass="10.0"/>
+        <visual>
+                <origin xyz="0 0 0" rpy="0 0 0"/>
+                <geometry>
+                        <mesh filename="file://$(find chandra_description)/meshes/base_link.STL" scale="${default_scale}"/>
+                </geometry>
+                <xacro:metallic_material name="base_link_material" colour="${deep_blue}"/>
+        </visual>
+        <collision>
+            <origin
+                    xyz="0 0 0"
+                    rpy="0 0 0"/>
+            <geometry>
+                <mesh
+                        filename="file://$(find chandra_description)/meshes/base_link.STL" scale="${default_scale}"/>
             </geometry>
         </collision>
     </link>
     <link name="link1">
-        <inertial>
-            <origin xyz="0 0 0" rpy="0 0 0"/>
-            <mass value="0.1"/>
-            <inertia ixx="0.0001" ixy="0.0" ixz="0.0" iyy="0.0001" iyz="0.0" izz="0.0001"/>
-        </inertial>
-        <visual>
-            <origin
-                    xyz="0 0 0"
-                    rpy="0 0 0"/>
-            <geometry>
-                <mesh
-                        filename="file://$(find chandra_description)/meshes/link1.STL"/>
-            </geometry>
-            <material
-                    name="">
-                <color
-                        rgba="0 0.7 0 1"/>
-            </material>
-        </visual>
-        <collision>
-            <origin
-                    xyz="0 0 0"
-                    rpy="0 0 0"/>
-            <geometry>
-                <mesh
-                        filename="file://$(find chandra_description)/meshes/link1.STL"/>
+        <xacro:default_inertial mass="2.0"/>
+        <visual>
+                <origin xyz="0 0 0" rpy="0 0 0"/>
+                <geometry>
+                        <mesh filename="file://$(find chandra_description)/meshes/link1.STL" scale="${default_scale}"/>
+                </geometry>
+                <xacro:metallic_material name="link1_material" colour="${green}"/>
+        </visual>
+        <collision>
+            <origin
+                    xyz="0 0 0"
+                    rpy="0 0 0"/>
+            <geometry>
+                <mesh
+                        filename="file://$(find chandra_description)/meshes/link1.STL" scale="${default_scale}"/>
             </geometry>
         </collision>
@@ -94,30 +86,19 @@
     </joint>
     <link name="link2">
-        <inertial>
-            <origin xyz="0 0 0" rpy="0 0 0"/>
-            <mass value="0.1"/>
-            <inertia ixx="0.0001" ixy="0.0" ixz="0.0" iyy="0.0001" iyz="0.0" izz="0.0001"/>
-        </inertial>
-        <visual>
-            <origin
-                    xyz="0 0 0"
-                    rpy="0 0 0"/>
-            <geometry>
-                <mesh
-                        filename="file://$(find chandra_description)/meshes/link2.STL"/>
-            </geometry>
-            <material
-                    name="">
-                <color
-                        rgba="0.7 0.7 0.7 1"/>
-            </material>
-        </visual>
-        <collision>
-            <origin
-                    xyz="0 0 0"
-                    rpy="0 0 0"/>
-            <geometry>
-                <mesh
-                        filename="file://$(find chandra_description)/meshes/link2.STL"/>
+        <xacro:default_inertial mass="1.5"/>
+        <visual>
+                <origin xyz="0 0 0" rpy="0 0 0"/>
+                <geometry>
+                        <mesh filename="file://$(find chandra_description)/meshes/link2.STL" scale="${default_scale}"/>
+                </geometry>
+                <xacro:metallic_material name="link2_material" colour="${deep_blue}"/>
+        </visual>
+        <collision>
+            <origin
+                    xyz="0 0 0"
+                    rpy="0 0 0"/>
+            <geometry>
+                <mesh
+                        filename="file://$(find chandra_description)/meshes/link2.STL" scale="${default_scale}"/>
             </geometry>
         </collision>
@@ -140,30 +121,19 @@
     </joint>
     <link name="link3">
-        <inertial>
-            <origin xyz="0 0 0" rpy="0 0 0"/>
-            <mass value="0.1"/>
-            <inertia ixx="0.0001" ixy="0.0" ixz="0.0" iyy="0.0001" iyz="0.0" izz="0.0001"/>
-        </inertial>
-        <visual>
-            <origin
-                    xyz="0 0 0"
-                    rpy="0 0 0"/>
-            <geometry>
-                <mesh
-                        filename="file://$(find chandra_description)/meshes/link3.STL"/>
-            </geometry>
-            <material
-                    name="">
-                <color
-                        rgba="0 0.7 0 1"/>
-            </material>
-        </visual>
-        <collision>
-            <origin
-                    xyz="0 0 0"
-                    rpy="0 0 0"/>
-            <geometry>
-                <mesh
-                        filename="file://$(find chandra_description)/meshes/link3.STL"/>
+        <xacro:default_inertial mass="1.0"/>
+        <visual>
+                <origin xyz="0 0 0" rpy="0 0 0"/>
+                <geometry>
+                        <mesh filename="file://$(find chandra_description)/meshes/link3.STL" scale="${default_scale}"/>
+                </geometry>
+                <xacro:metallic_material name="link3_material" colour="${green}"/>
+        </visual>
+        <collision>
+            <origin
+                    xyz="0 0 0"
+                    rpy="0 0 0"/>
+            <geometry>
+                <mesh
+                        filename="file://$(find chandra_description)/meshes/link3.STL" scale="${default_scale}"/>
             </geometry>
         </collision>
@@ -186,30 +156,19 @@
     </joint>
     <link name="link4">
-        <inertial>
-            <origin xyz="0 0 0" rpy="0 0 0"/>
-            <mass value="0.1"/>
-            <inertia ixx="0.0001" ixy="0.0" ixz="0.0" iyy="0.0001" iyz="0.0" izz="0.0001"/>
-        </inertial>
-        <visual>
-            <origin
-                    xyz="0 0 0"
-                    rpy="0 0 0"/>
-            <geometry>
-                <mesh
-                        filename="file://$(find chandra_description)/meshes/link4.STL"/>
-            </geometry>
-            <material
-                    name="">
-                <color
-                        rgba="0.7 0.7 0.7 1"/>
-            </material>
-        </visual>
-        <collision>
-            <origin
-                    xyz="0 0 0"
-                    rpy="0 0 0"/>
-            <geometry>
-                <mesh
-                        filename="file://$(find chandra_description)/meshes/link4.STL"/>
+        <xacro:default_inertial mass="0.7"/>
+        <visual>
+                <origin xyz="0 0 0" rpy="0 0 0"/>
+                <geometry>
+                        <mesh filename="file://$(find chandra_description)/meshes/link4.STL" scale="${default_scale}"/>
+                </geometry>
+                <xacro:metallic_material name="link4_material" colour="${deep_blue}"/>
+        </visual>
+        <collision>
+            <origin
+                    xyz="0 0 0"
+                    rpy="0 0 0"/>
+            <geometry>
+                <mesh
+                        filename="file://$(find chandra_description)/meshes/link4.STL" scale="${default_scale}"/>
             </geometry>
         </collision>
@@ -232,30 +191,19 @@
     </joint>
     <link name="link5">
-        <inertial>
-            <origin xyz="0 0 0" rpy="0 0 0"/>
-            <mass value="0.1"/>
-            <inertia ixx="0.0001" ixy="0.0" ixz="0.0" iyy="0.0001" iyz="0.0" izz="0.0001"/>
-        </inertial>
-        <visual>
-            <origin
-                    xyz="0 0 0"
-                    rpy="0 0 0"/>
-            <geometry>
-                <mesh
-                        filename="file://$(find chandra_description)/meshes/link5.STL"/>
-            </geometry>
-            <material
-                    name="">
-                <color
-                        rgba="1 1 1 1"/>
-            </material>
-        </visual>
-        <collision>
-            <origin
-                    xyz="0 0 0"
-                    rpy="0 0 0"/>
-            <geometry>
-                <mesh
-                        filename="file://$(find chandra_description)/meshes/link5.STL"/>
+        <xacro:default_inertial mass="0.5"/>
+        <visual>
+                <origin xyz="0 0 0" rpy="0 0 0"/>
+                <geometry>
+                        <mesh filename="file://$(find chandra_description)/meshes/link5.STL" scale="${default_scale}"/>
+                </geometry>
+                <xacro:metallic_material name="link5_material" colour="${deep_blue}"/>
+        </visual>
+        <collision>
+            <origin
+                    xyz="0 0 0"
+                    rpy="0 0 0"/>
+            <geometry>
+                <mesh
+                        filename="file://$(find chandra_description)/meshes/link5.STL" scale="${default_scale}"/>
             </geometry>
         </collision>
@@ -280,17 +228,16 @@
         <xacro:default_inertial mass="0.01"/>
         <visual>
+                <origin xyz="0.0121 0 -0.0335" rpy="0 0 0"/>
+                <geometry>
+                        <mesh filename="file://$(find chandra_description)/meshes/gripper_right_finger.STL" scale="${default_scale}"/>
+                </geometry>
+                <xacro:metallic_material name="gripper_right_material" colour="${black}"/>
+        </visual>
+        <collision>
             <origin
                     xyz="0.0121 0 -0.0335"
                     rpy="0 0 0"/>
             <geometry>
-                <mesh filename="file://$(find chandra_description)/meshes/gripper_right_finger.STL"/>
-            </geometry>
-        </visual>
-        <collision>
-            <origin
-                    xyz="0.0121 0 -0.0335"
-                    rpy="0 0 0"/>
-            <geometry>
-                <mesh filename="file://$(find chandra_description)/meshes/gripper_right_finger.STL"/>
+                <mesh filename="file://$(find chandra_description)/meshes/gripper_right_finger.STL" scale="${default_scale}"/>
             </geometry>
         </collision>
@@ -309,17 +256,16 @@
         <xacro:default_inertial mass="0.01"/>
         <visual>
+                <origin xyz="-0.0121 0 -0.0335" rpy="0 0 0"/>
+                <geometry>
+                        <mesh filename="file://$(find chandra_description)/meshes/gripper_left_finger.STL" scale="${default_scale}"/>
+                </geometry>
+                <xacro:metallic_material name="gripper_left_material" colour="${black}"/>
+        </visual>
+        <collision>
             <origin
                     xyz="-0.0121 0 -0.0335"
                     rpy="0 0 0"/>
             <geometry>
-                <mesh filename="file://$(find chandra_description)/meshes/gripper_left_finger.STL"/>
-            </geometry>
-        </visual>
-        <collision>
-            <origin
-                    xyz="-0.0121 0 -0.0335"
-                    rpy="0 0 0"/>
-            <geometry>
-                <mesh filename="file://$(find chandra_description)/meshes/gripper_left_finger.STL"/>
+                <mesh filename="file://$(find chandra_description)/meshes/gripper_left_finger.STL" scale="${default_scale}"/>
             </geometry>
         </collision>

Commit message: Add: Chandra moveit package

File: src/chandra_description/urdf/chandra_arm.urdf.xacro (robot description, xacro)
@@ -31,4 +31,10 @@
     <!-- Include ros2_control Plugins -->
     <xacro:include filename="$(find chandra_description)/urdf/chandra_arm_control.xacro" />
+    <link name="world"/>
+    <joint name="virtual_joint" type="fixed">
+        <parent link="world"/>
+        <child link="base_link"/>
+        <origin xyz="0 0 0" rpy="0 0 0"/>
+    </joint>
     <link name="base_link">
         <xacro:default_inertial mass="10.0"/>

File: src/chandra_description/urdf/chandra_arm_control.xacro (robot description, xacro)
@@ -1,6 +1,6 @@
 <?xml version="1.0"?>
 <robot xmlns:xacro="http://www.ros.org/wiki/xacro" name="chandra">
+    <xacro:property name="PI" value="3.14159265359" />
     <ros2_control name="RobotSystem" type="system">
-        <xacro:property name="PI" value="3.14159265359" />
         <hardware>
             <plugin>gz_ros2_control/GazeboSimSystem</plugin>

Commit message: Add: Real hardware interface

File: src/chandra_description/urdf/chandra_arm.urdf.xacro (robot description, xacro)
@@ -27,4 +27,5 @@
         </inertial>
     </xacro:macro>
+    <xacro:arg name="is_sim" default="False"/>
     <!-- Include Gazebo Parameters -->
     <xacro:include filename="$(find chandra_description)/urdf/chandra_arm_gazebo.xacro" />

File: src/chandra_description/urdf/chandra_arm_control.xacro (robot description, xacro)
@@ -3,8 +3,22 @@
     <xacro:property name="PI" value="3.14159265359" />
     <ros2_control name="RobotSystem" type="system">
-        <hardware>
-            <plugin>gz_ros2_control/GazeboSimSystem</plugin>
-        </hardware>
+        <!-- ros2_control Gazebo -->
+        <xacro:if value="$(arg is_sim)">
+            <hardware>
+                <plugin>gz_ros2_control/GazeboSimSystem</plugin>
+            </hardware>
+        <joint name="joint7">
+            <param name="mimic">joint6</param>
+            <param name="multiplier">-1</param>
+        </joint>
+        </xacro:if>
+        <!-- ros2_control Real Robot -->
+        <xacro:unless value="$(arg is_sim)">
+            <hardware>
+                <plugin>chandra_controller/ChandraInterface</plugin>
+            </hardware>
+        </xacro:unless>
         <joint name="joint1">
+            <param name="servo_id">1</param>
             <command_interface name="position">
             <param name="min">-${PI / 2}</param>
@@ -14,4 +28,5 @@
         </joint>
         <joint name="joint2">
+            <param name="servo_id">2</param>
             <command_interface name="position">
             <param name="min">-${PI / 2}</param>
@@ -21,4 +36,5 @@
         </joint>
         <joint name="joint3">
+            <param name="servo_id">3</param>
             <command_interface name="position">
             <param name="min">-${PI / 2}</param>
@@ -28,4 +44,5 @@
         </joint>
         <joint name="joint4">
+            <param name="servo_id">4</param>
             <command_interface name="position">
             <param name="min">-${PI / 2}</param>
@@ -35,4 +52,5 @@
         </joint>
         <joint name="joint5">
+            <param name="servo_id">5</param>
             <command_interface name="position">
             <param name="min">-${PI / 2}</param>
@@ -42,4 +60,5 @@
         </joint>
         <joint name="joint6">
+            <param name="servo_id">6</param>
             <command_interface name="position">
             <param name="min">-${PI / 2}</param>
@@ -48,8 +67,4 @@
             <state_interface name="position"/>
         </joint>
-        <joint name="joint7">
-            <param name="mimic">joint6</param>
-            <param name="multiplier">-1</param>
-        </joint>
     </ros2_control>
 </robot>

Commit message: Add:joint offsets

File: src/chandra_description/urdf/chandra_arm.urdf.xacro (robot description, xacro)
@@ -257,5 +257,5 @@
                 rpy="0 0 0"/>
         <axis xyz="0 1 0"/>
-        <limit lower="-${PI / 2}" upper="0.0"
+        <limit lower="-0.700" upper="0.807"
                effort="${effort}" velocity="${velocity}"/>
     </joint>
@@ -285,5 +285,5 @@
                 rpy="0 0 0"/>
         <axis xyz="0 1 0"/>
-        <limit lower="0.0" upper="${PI / 2}"
+        <limit lower="-0.807" upper="0.700"
                effort="${effort}" velocity="${velocity}"/>
         <mimic joint="joint6" multiplier="-1"/>
